File: flux_gate_3_axis.kicad_pcb (KiCad board)
At the start: 4 copper layers, 44 x 51.1 mm, 60 parts, among them J1 Conn_02x04_Odd_Even, J2 Conn_02x04_Odd_Even, J3 Conn_02x04_Odd_Even, J4 Conn_01x02, J5 Conn_01x02, J6 Conn_02x04_Odd_Even, J7 Conn_01x02, U1 Pico, U2 DRV425, U3 DRV425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

Commit message: added link to github repo
Other:
- board text added: "Magnetic field sensor (board B) v1.0 go.umd.edu/bsens"
- board text added: "Magnetic field sensor v1.0 (board A) Yanda Geng 2024.10 go.umd.edu/bsens"
- board text removed: "Magnetic field sensor (board B) v1.0"
- board text removed: "Magnetic field sensor v1.0 (board A) Yanda Geng 2024.10"
Changed lines of the file:
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@@
 		(tags "resistor")
 		(property "Reference" "R12"
-			(at 0 1.410441 360)
+			(at 0 1.410441 0)
 			(layer "F.SilkS")
 			(effects
@@
 		)
 		(property "Value" "24"
-			(at 0 1.65 360)
+			(at 0 1.65 0)
 			(layer "F.Fab")
 			(effects
@@
 		)
 		(property "Footprint" "Resistor_SMD:R_0805_2012Metric"
-			(at 0 0 360)
+			(at 0 0 0)
 			(layer "F.Fab")
 			(hide yes)
@@
 		)
 		(property "Datasheet" ""
-			(at 0 0 360)
+			(at 0 0 0)
 			(layer "F.Fab")
 			(hide yes)
@@
 		)
 		(property "Description" ""
-			(at 0 0 360)
+			(at 0 0 0)
 			(layer "F.Fab")
 			(hide yes)
@@
 		)
 		(fp_text user "${REFERENCE}"
-			(at 0 0 360)
+			(at 0 0 0)
 			(layer "F.Fab")
 			(effects
@@
 		)
 		(fp_text user "*"
-			(at -0.2 -1.2827 270)
+			(at -0.2 -1.2827 -90)
 			(unlocked yes)
 			(layer "F.SilkS")
@@
 		(tags "inductor")
 		(property "Reference" "L4"
-			(at 1.7 -0.05 360)
+			(at 1.7 -0.05 0)
 			(layer "F.SilkS")
 			(effects
@@
 		)
 		(property "Value" "BLM15AX601SN1D"
-			(at -5 0 360)
+			(at -5 0 0)
 			(layer "F.Fab")
 			(effects
@@
 		)
 		(fp_text user "${REFERENCE}"
-			(at 0 0 360)
+			(at 0 0 0)
 			(layer "F.Fab")
 			(effects
@@
 		(at 41.45 59.75 180)
 		(property "Reference" "G***"
-			(at 0 0 360)
+			(at 0 0 0)
 			(layer "B.SilkS")
 			(hide yes)
@@
 		)
 		(property "Value" "LOGO"
-			(at 0.75 0 360)
+			(at 0.75 0 0)
 			(layer "B.SilkS")
 			(hide yes)
@@
 		)
 		(property "Footprint" "flux_gate_footprints:JQI-Logo"
-			(at 0 0 360)
+			(at 0 0 0)
 			(layer "F.Fab")
 			(hide yes)
@@
 		)
 		(property "Datasheet" ""
-			(at 0 0 360)
+			(at 0 0 0)
 			(layer "F.Fab")
 			(hide yes)
@@
 		)
 		(property "Description" ""
-			(at 0 0 360)
+			(at 0 0 0)
 			(layer "F.Fab")
 			(hide yes)
@@
 		)
 	)
-	(gr_text "Magnetic field sensor\n(board B) v1.0"
-		(at 56.45 55.85 0)
+	(gr_text "Magnetic field sensor\n(board B) v1.0\ngo.umd.edu/bsens"
+		(at 56.45 56.05 0)
 		(layer "B.SilkS")
 		(effects
@@
 		)
 	)
-	(gr_text "Magnetic field sensor v1.0\n(board A)\nYanda Geng 2024.10"
-		(at 41.95 15.55 90)
+	(gr_text "Magnetic field sensor v1.0\n(board A)\nYanda Geng 2024.10\ngo.umd.edu/bsens"
+		(at 38.35 15.55 90)
 		(layer "B.SilkS")
 		(effects
@@
 				(thickness 0.15)
 			)
-			(justify left bottom mirror)
+			(justify left top mirror)
 		)
 	)
